File: power.kicad_sch (KiCad schematic)
At the start: 14 parts, among them J1 Conn_01x04, J2 Conn_01x04

Commit message: Remove everything not needed for JTAG loader board testing
Parts:
- removed H1, H2, H5, H6, H7, H8: MountingHole_Pad, MountingHole:MountingHole_3.2mm_M3_DIN965_Pad, symbol Mechanical:MountingHole_Pad
