File: multiplexorbus.kicad_sch (KiCad schematic)
At the start: 8 parts, among them J10 PMOD2, J11 Conn_02x05_Odd_Even, J12 Conn_02x17_Odd_Even, J13 Conn_02x17_Odd_Even, J15 ESP32 Connector, J7 Conn_02x06_Odd_Even, J8 Conn_02x06_Odd_Even, J9 PMOD1

Commit message: Remove everything not needed for JTAG loader board testing
Parts:
- removed J11: Conn_02x05_Odd_Even, Connector_PinHeader_2.54mm:PinHeader_2x05_P2.54mm_Vertical, symbol Connector_Generic:Conn_02x05_Odd_Even
- removed J7: Conn_02x06_Odd_Even, Connector_PinHeader_2.54mm:PinHeader_2x06_P2.54mm_Vertical, symbol Connector_Generic:Conn_02x06_Odd_Even
Connections:
- no-connect marks 9 -> 5

Commit message: Minor changes from DRC.
Parts:
- added J14: Conn_02x05_Odd_Even, Connector_PinHeader_2.54mm:PinHeader_2x05_P2.54mm_Vertical, symbol Connector_Generic:Conn_02x05_Odd_Even
- added J7: Conn_02x06_Odd_Even, Connector_PinHeader_2.54mm:PinHeader_2x06_P2.54mm_Vertical, symbol Connector_Generic:Conn_02x06_Odd_Even
Connections:
- net TE0790_10: now also J14.9 (Pin_9), J7.10 (Pin_10)
- net TE0790_12: now also J14.5 (Pin_5), J7.12 (Pin_12)
- net TE0790_2: now also J14.2 (Pin_2), J7.2 (Pin_2)
- net TE0790_3: now also J14.7 (Pin_7), J7.3 (Pin_3)
- net TE0790_4: now also J14.1 (Pin_1), J7.4 (Pin_4)
- net TE0790_6: now also J14.4 (Pin_4), J7.6 (Pin_6)
- net TE0790_7: now also J14.8 (Pin_8), J7.7 (Pin_7)
- net TE0790_8: now also J14.3 (Pin_3), J7.8 (Pin_8)
- no-connect marks 5 -> 9

Commit message: Add in the temodule and the step layers
Parts:
- J10, J9: footprint Connector_PinHeader_2.54mm:PinHeader_2x06_P2.54mm_Vertical -> Connector_PinSocket_2.54mm:PinSocket_2x06_P2.54mm_Horizontal
Changed lines of the file:
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@@
 			)
 		)
-		(property "Footprint" "Connector_PinHeader_2.54mm:PinHeader_2x06_P2.54mm_Vertical"
+		(property "Footprint" "Connector_PinSocket_2.54mm:PinSocket_2x06_P2.54mm_Horizontal"
 			(at 77.47 45.72 0)
 			(hide yes)
@@
 			)
 		)
-		(property "Footprint" "Connector_PinHeader_2.54mm:PinHeader_2x06_P2.54mm_Vertical"
+		(property "Footprint" "Connector_PinSocket_2.54mm:PinSocket_2x06_P2.54mm_Horizontal"
 			(at 77.47 80.01 0)
 			(hide yes)
